Commit message: for colab

File: darwin_gym/darwin_gym/envs/darwin2.urdf (robot description, URDF)
Before this commit: robot darwinOP, 30 links, 29 joints
Links:
- link MP_ANKLE1_L: geometry collision mesh filename=/content/DarwinOp_gym/darwin_gym/darwin_gym/envs/meshes/ank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 scale=1 1 1; visual mesh filename=/content/DarwinOp_gym/darwin_gym/darwin_gym/envs/meshes/ank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 scale=1 1 1
- link MP_ANKLE1_R: geometry collision mesh filename=/content/DarwinOp_gym/darwin_gym/darwin_gym/envs/meshes/ank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 scale=1 1 1; visual mesh filename=/content/DarwinOp_gym/darwin_gym/darwin_gym/envs/meshes/ank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 scale=1 1 1
- link MP_ANKLE2_L: geometry collision mesh filename=/content/DarwinOp_gym/darwin_gym/darwin_gym/envs/meshes/ank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 scale=1 1 1; visual mesh filename=/content/DarwinOp_gym/darwin_gym/darwin_gym/envs/meshes/ank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 scale=1 1 1
- link MP_ANKLE2_R: geometry collision mesh filename=/content/DarwinOp_gym/darwin_gym/darwin_gym/envs/meshes/ank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 scale=1 1 1; visual mesh filename=/content/DarwinOp_gym/darwin_gym/darwin_gym/envs/meshes/ank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 scale=1 1 1
- link MP_ARM_HIGH_L: geometry collision mesh filename=/content/DarwinOp_gym/darwin_gym/darwin_gym/envs/meshes/arm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 scale=1 1 1; visual mesh filename=/content/DarwinOp_gym/darwin_gym/darwin_gym/envs/meshes/arm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 scale=1 1 1
- link MP_ARM_HIGH_R: geometry collision mesh filename=/content/DarwinOp_gym/darwin_gym/darwin_gym/envs/meshes/arm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 scale=1 1 1; visual mesh filename=/content/DarwinOp_gym/darwin_gym/darwin_gym/envs/meshes/arm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 scale=1 1 1
- link MP_BODY: geometry collision mesh filename=/content/DarwinOp_gym/darwin_gym/darwin_gym/envs//content/D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 scale=1 1 1; visual mesh filename=/content/DarwinOp_gym/darwin_gym/darwin_gym/envs/meshes/bod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 scale=1 1 1
- link MP_HEAD: geometry collision mesh filename=/content/DarwinOp_gym/darwin_gym/darwin_gym/envs/meshes/hea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 scale=1 1 1; visual mesh filename=/content/DarwinOp_gym/darwin_gym/darwin_gym/envs/meshes/hea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 scale=1 1 1
- link MP_NECK: geometry collision mesh filename=/content/DarwinOp_gym/darwin_gym/darwin_gym/envs/meshes/nec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 scale=1 1 1; visual mesh filename=/content/DarwinOp_gym/darwin_gym/darwin_gym/envs//content/D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 scale=1 1 1
- link MP_PELVIS_L: geometry collision mesh filename=/content/DarwinOp_gym/darwin_gym/darwin_gym/envs/meshes/pel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 scale=1 1 1; visual mesh filename=/content/DarwinOp_gym/darwin_gym/darwin_gym/envs/meshes/pel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 scale=1 1 1
- link MP_PELVIS_R: geometry collision mesh filename=/content/DarwinOp_gym/darwin_gym/darwin_gym/envs/meshes/pel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 scale=1 1 1; visual mesh filename=/content/DarwinOp_gym/darwin_gym/darwin_gym/envs/meshes/pel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 scale=1 1 1
- link MP_SHOULDER_L: geometry collision mesh filename=/content/DarwinOp_gym/darwin_gym/darwin_gym/envs/meshes/sho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 scale=1 1 1; visual mesh filename=/content/DarwinOp_gym/darwin_gym/darwin_gym/envs/meshes/sho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 scale=1 1 1
- link MP_SHOULDER_R: geometry collision mesh filename=/content/DarwinOp_gym/darwin_gym/darwin_gym/envs/meshes/sho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 scale=1 1 1; visual mesh filename=/content/DarwinOp_gym/darwin_gym/darwin_gym/envs/meshes/sho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 scale=1 1 1
- link MP_THIGH1_L: geometry collision mesh filename=/content/DarwinOp_gym/darwin_gym/darwin_gym/envs/meshes/thi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 scale=1 1 1; visual mesh filename=/content/DarwinOp_gym/darwin_gym/darwin_gym/envs/meshes/thi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 scale=1 1 1
- link MP_THIGH1_R: geometry collision mesh filename=/content/DarwinOp_gym/darwin_gym/darwin_gym/envs/meshes/thi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 scale=1 1 1; visual mesh filename=/content/DarwinOp_gym/darwin_gym/darwin_gym/envs/meshes/thi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 scale=1 1 1
- link MP_THIGH2_L: geometry collision mesh filename=/content/DarwinOp_gym/darwin_gym/darwin_gym/envs/meshes/thi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 scale=1 1 1; visual mesh filename=/content/DarwinOp_gym/darwin_gym/darwin_gym/envs/meshes/thi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 scale=1 1 1
- link MP_THIGH2_R: geometry collision mesh filename=/content/DarwinOp_gym/darwin_gym/darwin_gym/envs/meshes/thi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 scale=1 1 1; visual mesh filename=/content/DarwinOp_gym/darwin_gym/darwin_gym/envs/meshes/thi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 scale=1 1 1
- link MP_TIBIA_L: geometry collision mesh filename=/content/DarwinOp_gym/darwin_gym/darwin_gym/envs/meshes/tib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 scale=1 1 1; visual mesh filename=/content/DarwinOp_gym/darwin_gym/darwin_gym/envs/meshes/tib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 scale=1 1 1
- link MP_TIBIA_R: geometry collision mesh filename=/content/DarwinOp_gym/darwin_gym/darwin_gym/envs/meshes/tib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 scale=1 1 1; visual mesh filename=/content/DarwinOp_gym/darwin_gym/darwin_gym/envs/meshes/tib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 scale=1 1 1

Commit message: urdf corrected

File: darwin_gym/darwin_gym/envs/darwin2.urdf (robot description, URDF)
Before this commit: robot darwinOP, 30 links, 29 joints
Links:
- link MP_BODY: geometry collision mesh filename=/content/DarwinOp_gym/darwin_gym/darwin_gym/envs/meshes/bod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 scale=1 1 1; visual mesh filename=/content/DarwinOp_gym/darwin_gym/darwin_gym/envs/meshes/bod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 scale=1 1 1
- link MP_NECK: geometry collision mesh filename=/content/DarwinOp_gym/darwin_gym/darwin_gym/envs/meshes/nec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 scale=1 1 1; visual mesh filename=/content/DarwinOp_gym/darwin_gym/darwin_gym/envs/meshes/nec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 scale=1 1 1

Commit message: realtimesim line deleted and ankle off

File: darwin_gym/darwin_gym/envs/darwin2.urdf (robot description, URDF)
Before this commit: robot darwinOP, 30 links, 29 joints
Joints:
- removed joint j_ankle1_l
- removed joint j_ankle1_r
- removed joint j_ankle2_l
- removed joint j_ankle2_r
- added joint jointfixj_ankle1_l: type revolute, parent MP_TIBIA_L, child MP_ANKLE1_L, origin xyz=-0.093 0 0 rpy=3.14159 0 0, axis 0 0 1, limit lower=-2.6179939 upper=2.6179939 effort=10 velocity=5.6548668
- added joint jointfixj_ankle1_r: type revolute, parent MP_TIBIA_R, child MP_ANKLE1_R, origin xyz=0.093 0 0 rpy=3.14159 0 0, axis 0 0 1, limit lower=-2.6179939 upper=2.6179939 effort=10 velocity=5.6548668
- added joint jointfixj_ankle2_l: type revolute, parent MP_ANKLE1_L, child MP_ANKLE2_L, origin xyz=0 0 0 rpy=-1.5707963 0 0, axis 0 0 1, limit lower=-2.6179939 upper=2.6179939 effort=10 velocity=5.6548668
- added joint jointfixj_ankle2_r: type revolute, parent MP_ANKLE1_R, child MP_ANKLE2_R, origin xyz=0 0 0 rpy=-1.5707963 0 0, axis 0 0 1, limit lower=-2.6179939 upper=2.6179939 effort=10 velocity=5.6548668

Commit message: urdf changed joint limits reduced

File: darwin_gym/darwin_gym/envs/darwin2.urdf (robot description, URDF)
Before this commit: robot darwinOP, 30 links, 29 joints
Joints:
- removed joint jointfixj_ankle1_l
- removed joint jointfixj_ankle1_r
- removed joint jointfixj_ankle2_l
- removed joint jointfixj_ankle2_r
- added joint j_ankle1_l: type revolute, parent MP_TIBIA_L, child MP_ANKLE1_L, origin xyz=-0.093 0 0 rpy=3.14159 0 0, axis 0 0 1, limit lower=-0.26179939 upper=.26179939 effort=10 velocity=5.6548668
- added joint j_ankle1_r: type revolute, parent MP_TIBIA_R, child MP_ANKLE1_R, origin xyz=0.093 0 0 rpy=3.14159 0 0, axis 0 0 1, limit lower=-0.26179939 upper=0.26179939 effort=10 velocity=5.6548668
- added joint j_ankle2_l: type revolute, parent MP_ANKLE1_L, child MP_ANKLE2_L, origin xyz=0 0 0 rpy=-1.5707963 0 0, axis 0 0 1, limit lower=-.26179939 upper=.26179939 effort=10 velocity=5.6548668
- added joint j_ankle2_r: type revolute, parent MP_ANKLE1_R, child MP_ANKLE2_R, origin xyz=0 0 0 rpy=-1.5707963 0 0, axis 0 0 1, limit lower=-0.26179939 upper=0.26179939 effort=10 velocity=5.6548668
- joint j_high_arm_l: limit lower=-2.6179939 upper=2.6179939 effort=2.8 velocity=5.648668 -> lower=-0.7179939 upper=1.8179939 effort=2.8 velocity=5.648668
- joint j_high_arm_r: limit lower=-2.6179939 upper=2.6179939 effort=2.8 velocity=5.648668 -> lower=-0.7179939 upper=1.8179939 effort=2.8 velocity=5.648668
- joint j_low_arm_l: limit lower=-2.6179939 upper=2.6179939 effort=2.8 velocity=5.6548668 -> lower=-2.6179939 upper=0.635 effort=2.8 velocity=5.6548668
- joint j_low_arm_r: limit lower=-1.635 upper=2.6179939 effort=2.8 velocity=5.6548668 -> lower=-0.635 upper=2.6179939 effort=2.8 velocity=5.6548668
- joint j_pelvis_l: limit lower=-2.6179939 upper=2.6179939 effort=10 velocity=5.6548668 -> lower=-0.6179939 upper=0.6179939 effort=10 velocity=5.6548668
- joint j_pelvis_r: limit lower=-2.6179939 upper=2.6179939 effort=10 velocity=5.6548668 -> lower=-0.6179939 upper=0.6179939 effort=10 velocity=5.6548668
- joint j_shoulder_l: limit lower=-2.6179939 upper=2.6179939 effort=2.8 velocity=5.6548668 -> lower=-9.8179939 upper=0.9179939 effort=2.8 velocity=5.6548668
- joint j_shoulder_r: limit lower=-2.6179939 upper=2.6179939 effort=2.8 velocity=5.6548668 -> lower=-0.9179939 upper=0.9179939 effort=2.8 velocity=5.6548668
- joint j_thigh1_l: limit lower=-2.6179939 upper=2.6179939 effort=10 velocity=5.6548668 -> lower=-.6179939 upper=0.06179939 effort=10 velocity=5.6548668
- joint j_thigh1_r: limit lower=-2.6179939 upper=2.6179939 effort=10 velocity=5.6548668 -> lower=-0.06179939 upper=0.6179939 effort=10 velocity=5.6548668
- joint j_thigh2_l: limit lower=-2.6179939 upper=2.6179939 effort=10 velocity=5.6548668 -> lower=-0.6179939 upper=1.3179939 effort=10 velocity=5.6548668
- joint j_thigh2_r: limit lower=-2.6179939 upper=2.6179939 effort=10 velocity=5.6548668 -> lower=-1.3179939 upper=0.6179939 effort=10 velocity=5.6548668
- joint j_tibia_l: limit lower=-2.6179939 upper=2.6179939 effort=10 velocity=5.6548668 -> lower=-1.8879939 upper=0.06179939 effort=10 velocity=5.6548668
- joint j_tibia_r: limit lower=-2.6179939 upper=2.6179939 effort=10 velocity=5.6548668 -> lower=-0.06179939 upper=1.8879939 effort=10 velocity=5.6548668
