Commit message: added ankles

File: darwin_gym/darwin_gym/envs/darwin4.urdf (robot description, URDF)
Before this commit: robot darwinOP, 30 links, 29 joints
Joints:
- removed joint jointfixj_ankle1_l
- removed joint jointfixj_ankle1_r
- removed joint jointfixj_ankle2_l
- removed joint jointfixj_ankle2_r
- added joint j_ankle1_l: type revolute, parent MP_TIBIA_L, child MP_ANKLE1_L, origin xyz=-0.093 0 0 rpy=3.14159 0 0, axis 0 0 1, limit lower=-0.26179939 upper=.26179939 effort=10 velocity=5.6548668
- added joint j_ankle1_r: type revolute, parent MP_TIBIA_R, child MP_ANKLE1_R, origin xyz=0.093 0 0 rpy=3.14159 0 0, axis 0 0 1, limit lower=-0.26179939 upper=0.26179939 effort=10 velocity=5.6548668
- added joint j_ankle2_l: type revolute, parent MP_ANKLE1_L, child MP_ANKLE2_L, origin xyz=0 0 0 rpy=-1.5707963 0 0, axis 0 0 1, limit lower=-.26179939 upper=.26179939 effort=10 velocity=5.6548668
- added joint j_ankle2_r: type revolute, parent MP_ANKLE1_R, child MP_ANKLE2_R, origin xyz=0 0 0 rpy=-1.5707963 0 0, axis 0 0 1, limit lower=-0.26179939 upper=0.26179939 effort=10 velocity=5.6548668

Commit message: Branch for local changes

File: darwin_gym/darwin_gym/envs/darwin4.urdf (robot description, URDF)
Before this commit: robot darwinOP, 30 links, 29 joints
Links:
- link MP_ANKLE1_L: geometry collision mesh filename=/home/akash/Documents/RLcontrol/DarwinOp_gym/darwin_gym/dar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 scale=1 1 1; visual mesh filename=/home/akash/Documents/RLcontrol/DarwinOp_gym/darwin_gym/dar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 scale=1 1 1
- link MP_ANKLE1_R: geometry collision mesh filename=/home/akash/Documents/RLcontrol/DarwinOp_gym/darwin_gym/dar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 scale=1 1 1; visual mesh filename=/home/akash/Documents/RLcontrol/DarwinOp_gym/darwin_gym/dar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 scale=1 1 1
- link MP_ANKLE2_L: geometry collision mesh filename=/home/akash/Documents/RLcontrol/DarwinOp_gym/darwin_gym/dar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 scale=1 1 1; visual mesh filename=/home/akash/Documents/RLcontrol/DarwinOp_gym/darwin_gym/dar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 scale=1 1 1
- link MP_ANKLE2_R: geometry collision mesh filename=/home/akash/Documents/RLcontrol/DarwinOp_gym/darwin_gym/dar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 scale=1 1 1; visual mesh filename=/home/akash/Documents/RLcontrol/DarwinOp_gym/darwin_gym/dar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 scale=1 1 1
- link MP_ARM_HIGH_L: geometry collision mesh filename=/home/akash/Documents/RLcontrol/DarwinOp_gym/darwin_gym/dar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 scale=1 1 1; visual mesh filename=/home/akash/Documents/RLcontrol/DarwinOp_gym/darwin_gym/dar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 scale=1 1 1
- link MP_ARM_HIGH_R: geometry collision mesh filename=/home/akash/Documents/RLcontrol/DarwinOp_gym/darwin_gym/dar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 scale=1 1 1; visual mesh filename=/home/akash/Documents/RLcontrol/DarwinOp_gym/darwin_gym/dar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 scale=1 1 1
- link MP_BODY: geometry collision mesh filename=/home/akash/Documents/RLcontrol/DarwinOp_gym/darwin_gym/dar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 scale=1 1 1; visual mesh filename=/home/akash/Documents/RLcontrol/DarwinOp_gym/darwin_gym/dar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 scale=1 1 1
- link MP_HEAD: geometry collision mesh filename=/home/akash/Documents/RLcontrol/DarwinOp_gym/darwin_gym/dar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 scale=1 1 1; visual mesh filename=/home/akash/Documents/RLcontrol/DarwinOp_gym/darwin_gym/dar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 scale=1 1 1
- link MP_NECK: geometry collision mesh filename=/home/akash/Documents/RLcontrol/DarwinOp_gym/darwin_gym/dar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 scale=1 1 1; visual mesh filename=/home/akash/Documents/RLcontrol/DarwinOp_gym/darwin_gym/dar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 scale=1 1 1
- link MP_PELVIS_L: geometry collision mesh filename=/home/akash/Documents/RLcontrol/DarwinOp_gym/darwin_gym/dar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 scale=1 1 1; visual mesh filename=/home/akash/Documents/RLcontrol/DarwinOp_gym/darwin_gym/dar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 scale=1 1 1
- link MP_PELVIS_R: geometry collision mesh filename=/home/akash/Documents/RLcontrol/DarwinOp_gym/darwin_gym/dar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 scale=1 1 1; visual mesh filename=/home/akash/Documents/RLcontrol/DarwinOp_gym/darwin_gym/dar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 scale=1 1 1
- link MP_SHOULDER_L: geometry collision mesh filename=/home/akash/Documents/RLcontrol/DarwinOp_gym/darwin_gym/dar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 scale=1 1 1; visual mesh filename=/home/akash/Documents/RLcontrol/DarwinOp_gym/darwin_gym/dar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 scale=1 1 1
- link MP_SHOULDER_R: geometry collision mesh filename=/home/akash/Documents/RLcontrol/DarwinOp_gym/darwin_gym/dar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 scale=1 1 1; visual mesh filename=/home/akash/Documents/RLcontrol/DarwinOp_gym/darwin_gym/dar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 scale=1 1 1
- link MP_THIGH1_L: geometry collision mesh filename=/home/akash/Documents/RLcontrol/DarwinOp_gym/darwin_gym/dar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 scale=1 1 1; visual mesh filename=/home/akash/Documents/RLcontrol/DarwinOp_gym/darwin_gym/dar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 scale=1 1 1
- link MP_THIGH1_R: geometry collision mesh filename=/home/akash/Documents/RLcontrol/DarwinOp_gym/darwin_gym/dar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 scale=1 1 1; visual mesh filename=/home/akash/Documents/RLcontrol/DarwinOp_gym/darwin_gym/dar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 scale=1 1 1
- link MP_THIGH2_L: geometry collision mesh filename=/home/akash/Documents/RLcontrol/DarwinOp_gym/darwin_gym/dar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 scale=1 1 1; visual mesh filename=/home/akash/Documents/RLcontrol/DarwinOp_gym/darwin_gym/dar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 scale=1 1 1
- link MP_THIGH2_R: geometry collision mesh filename=/home/akash/Documents/RLcontrol/DarwinOp_gym/darwin_gym/dar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 scale=1 1 1; visual mesh filename=/home/akash/Documents/RLcontrol/DarwinOp_gym/darwin_gym/dar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 scale=1 1 1
- link MP_TIBIA_L: geometry collision mesh filename=/home/akash/Documents/RLcontrol/DarwinOp_gym/darwin_gym/dar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 scale=1 1 1; visual mesh filename=/home/akash/Documents/RLcontrol/DarwinOp_gym/darwin_gym/dar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 scale=1 1 1
- link MP_TIBIA_R: geometry collision mesh filename=/home/akash/Documents/RLcontrol/DarwinOp_gym/darwin_gym/dar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 scale=1 1 1; visual mesh filename=/home/akash/Documents/RLcontrol/DarwinOp_gym/darwin_gym/dar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 scale=1 1 1
